File: chickensticks.kicad_pcb (KiCad board)
At the start: 4 copper layers, 42 x 100 mm, 97 parts, among them J1 Conn_01x05_Pin, J2 HRO_TYPE-C-31-M-12, J3 Conn_01x04, J4 Conn_01x06, J5 Conn_01x06, J6 Conn_01x04, J7 Conn_01x04, J8 S02-25200300, J9 SMA, Q1 Si2371EDS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

Commit message: Implement first stage of review fixes
Parts:
- moved C25 3.76 mm to (118.8, 94.8), turned to 90 degrees
- moved C15 1.45 mm to (129.5, 95.8), turned to -90 degrees
- moved C14 0.94 mm to (127.5, 95.5), turned to -90 degrees
- moved Y2 0.86 mm to (116.5, 95.1)
- moved C12 0.11 mm to (117.3, 92.1)
Routing:
- net GND: track 4.22 -> 0.54 mm, vias 506 -> 733
- net Net-(U4-VDCC1): track 15.7 -> 17.8 mm
- net Net-(Q1-G): track 3.67 -> 4.69 mm
- net Net-(U4-VPAX1): track 11.5 -> 12.3 mm
- net Net-(U4-XTA): track 4.69 -> 5.49 mm

Commit message: Add buzzer, fix some erc
Parts:
- added BZ1: MLT-7525, Library:MLT-7525, B.Cu at (125.4, 145.7)
- added D12: 1N4148, APRLPrints:SOD-323, F.Cu at (126.5, 143.7)
- added Q3: 2N7002, Package_TO_SOT_SMD:SOT-23, F.Cu at (126.6, 140.7)
- added R19: 10k, APRLPrints:R_0603, F.Cu at (123.6, 141.9)
- added R20: 100R, APRLPrints:R_0603, F.Cu at (123.6, 139.1)
Connections:
- U2 pad 29: unconnected-(U2-PA8-Pad29) -> /Microcontroller/BUZZER
Routing:
- net /Microcontroller/BUZZER: track 0.00 -> 34.1 mm, vias 0 -> 2
- net +VUSB: track 29.4 -> 48.5 mm, vias 7 -> 8
- net Net-(BZ1--): track 0.00 -> 15.9 mm, vias 0 -> 1
- net Net-(Q3-G): track 0.00 -> 3.50 mm
- net GND: vias 733 -> 738

Commit message: Run cleanup tracks and vias
Routing:
- net /Microcontroller/~{RST}: track 18.1 -> 17.1 mm
- net +VUSB: track 48.5 -> 47.7 mm
- net /Microcontroller/ENC_C: track 42.0 -> 41.3 mm
- net /Microcontroller/CANL: track 7.24 -> 6.68 mm
- net Net-(J2-CC2): track 3.17 -> 2.62 mm

Commit message: Remove big SS14 diodes
Parts:
- removed the D1 at (117.4, 131.3)
- C7: moved to F.Cu
- D1: renamed from D5; value SS14 -> MM3Z10VT1G; footprint Diode_SMD:D_SMA -> APRLPrints:SOD-323
- moved D9 4.78 mm to (114.2, 125.7)
- moved C7 2.97 mm to (114.5, 133.3)
- moved R11 1.40 mm to (114.2, 128.5), turned to 90 degrees
- moved F1 1.33 mm to (117.4, 134.7), turned to 90 degrees
Connections:
- F1 pad 2: Net-(D1-A) (its old number) -> +VUSB
Routing:
- net Net-(D1-A): track 13.7 -> 14.5 mm
- net Net-(D9-A): track 2.20 -> 1.47 mm
- net +VUSB: track 47.7 -> 47.2 mm, vias 8 -> 5
- net GND: vias 738 -> 757
- removed copper zone on B.Cu, net +VUSB
- removed copper zone on F.Cu, net Net-(D1-A) (its old number)

Commit message: Add external 3.3V selector (noise is not real anyway)
Parts:
- removed D12: 1N4148, APRLPrints:SOD-323
- added D5: MM3Z10VT1G, APRLPrints:SOD-323, F.Cu at (126.4, 143.7)
- added J10: Conn_01x03_Pin, Connector_PinHeader_2.54mm:PinHeader_1x03_P2.54mm_Vertical, F.Cu at (112.5, 110.0)
- moved C31 4.01 mm to (116.2, 107.5)
- moved C29 3.99 mm to (116.2, 103.5)
- moved D10 1.78 mm to (110.9, 101.6), turned to -90 degrees
- moved R12 0.45 mm to (113.2, 102.2)
Connections:
- J1 pad 2: unconnected-(J1-Pin_2-Pad2) -> +3.3V_EXT
- U5 pad 5: +3.3V -> /Power/3.3_LDO_OUT
Routing:
- net GND: vias 757 -> 751
- added copper zone on In2.Cu, net +3.3V_EXT
- added copper zone on F.Cu, net /Power/3.3_LDO_OUT
